File: lmc_media_blitz.kicad_sch (KiCad schematic)
At the start: 40 parts, among them J3 Conn_ARM_JTAG_SWD_10, Q1 2N7002, Q2 2N7002, U1 TPS61222DCK, U2 XC6206PxxxMR, U5 LPC804M101JHI33

Commit message: Added STM32 MCU with prelim pinout to the schematic
Parts:
- added C41, C42, C43: 100nF, Capacitor_SMD:C_0603_1608Metric, symbol Device:C
- added C44: 10uF, Capacitor_SMD:C_0805_2012Metric, symbol Device:C
- added C45: 10nF, Capacitor_SMD:C_0603_1608Metric, symbol Device:C
- added C46: 1uF, Capacitor_SMD:C_0805_2012Metric, symbol Device:C
- added C47: 22uF, Capacitor_SMD:C_0805_2012Metric, symbol Device:C_Small
- added D7: SSL54B, Diode_SMD:D_SMB, symbol Device:D_Schottky_Small_Filled
- added L4: 4u7, Inductor_SMD:L_Sunlord_SWPA6045S, symbol Device:L_Small
- added Q3: BSS138W, PCM_JLCPCB:Q_SOT-323, symbol PCM_JLCPCB-Transistors:NMOS,BSS138W
- added Q4: BSS138, Package_TO_SOT_SMD:SOT-23, symbol Transistor_FET:BSS138
- added U15: TPS613222ADBV, Package_TO_SOT_SMD:SOT-23-5, symbol Regulator_Switching:TPS613222ADBV
- added U3: STM32F030C8Tx, Package_QFP:LQFP-48_7x7mm_P0.5mm, symbol MCU_ST_STM32F0:STM32F030C8Tx
- C5: value 0.1uF -> 100nF
Connections:
- net +3V3: now also C41.1, C42.1, C43.1, C44.2, C45.1, C46.1, U3.1 (VDD), U3.24 (VDD), U3.48 (VDD), U3.9 (VDDA)
- net +BATT: now also U3.10 (PA0); no longer C1.2
- net GND: now also C41.2, C42.2, C43.2, C44.1, C45.2, C46.2, C47.2, U15.2 (GND), U3.23 (VSS), U3.47 (VSS), U3.8 (VSSA)
- net SPI0_MOSI: now also U3.17 (PA7)
- net SPI0_SCKB: no longer Q2.1 (G), Q2.2 (S), R5.2
- net SWCLK: now also U3.37 (PA14)
- net SWDIO: now also U3.34 (PA13)
- new net: C47.1, D7.1 (K), U15.4 (VOUT)
- new net: C1.2, L4.1
- new net BOOST_SW: D7.2 (A), L4.2, U15.1 (SW)
- new net GPIO_EXTI10: U3.21 (PB10)
- new net I2C1_SCL: U3.42 (PB6)
- new net I2C1_SDA: U3.43 (PB7)
- new net SPI1_MISO: U3.16 (PA6)
- new net SPI1_SCK: Q2.1 (G), Q2.2 (S), R5.2, U3.15 (PA5)
- new net SPI2_MISO: U3.27 (PB14)
- new net SPI2_MOSI: U3.28 (PB15)
- new net SPI2_NSS: U3.25 (PB12)
- new net SPI2_SCK: U3.26 (PB13)
- new net SW1: U3.45 (PB8)
- new net SW2: U3.46 (PB9)
- new net SW3: U3.2 (PC13)
- new net USART1_RX: U3.31 (PA10)
- new net USART1_TX: U3.30 (PA9)
- new net nRST: U3.7 (NRST)
- no-connect marks 15 -> 34
Other:
- note added: "Boost Converter (1V5 -> 5V)"
- moved on the sheet: C1, TP1

Commit message: Added pushbutton part to schematic
Parts:
- removed C47: 22uF, Capacitor_SMD:C_0805_2012Metric, symbol Device:C_Small
- added C47, C49: 100nF, Capacitor_SMD:C_0603_1608Metric, symbol Device:C
- added C48: 22uF, Capacitor_SMD:C_0805_2012Metric, symbol Device:C
- added R10, R11: 10K, Resistor_SMD:R_0805_2012Metric, symbol Device:R
- added SW1, SW2: SW_Push, Button_Switch_SMD:SW_Push_1P1T_XKB_TS-1187A, symbol Switch:SW_Push
- C39: value 0.1uF -> 100nF
- L4: footprint Inductor_SMD:L_Sunlord_SWPA6045S -> Inductor_SMD:L_Changjiang_FNR4030S; LCSC Part # C78804 -> C167874
Connections:
- net +3V3: now also R10.1, R11.1
- net GND: now also C48.1
- net at D7.1 (K), U15.4 (VOUT): now also C48.2
- new net: C49.1, R11.2, SW2.2
- new net: C47.2, SW1.1
- new net: C47.1, R10.2, SW1.2
- new net: C49.2, SW2.1

Commit message: Placed 2 1x10 pin headers.  Pinout TBD
Parts:
- added C50: 100nF, Capacitor_SMD:C_0603_1608Metric, symbol Device:C
- added J4, J5: Conn_01x10, Connector_PinHeader_2.54mm:PinHeader_1x10_P2.54mm_Vertical, symbol Connector_Generic:Conn_01x10
- added R12: 10K, Resistor_SMD:R_0805_2012Metric, symbol Device:R
- added SW3: SW_Push, Button_Switch_SMD:SW_Push_1P1T_XKB_TS-1187A, symbol Switch:SW_Push
Connections:
- net +3V3: now also R12.1
- net SW1: now also C47.1, R10.2, SW1.2
- net SW2: now also C49.1, R11.2, SW2.2
- net SW3: now also C50.1, R12.2, SW3.2
- new net: C50.2, SW3.1
Other:
- note added: "PN532, MFRC522 both support 3V3 SPI, I2C, UART PN532 can run off 5V supply, both can be powered with 3V3"
- moved on the sheet: C41, C42, C43, C44, C45, C46, C47, R10, SW1, U3

Commit message: Wired up 5V boost, 3V3 LDO, and power to STM32 MCU
Parts:
- removed C38, C44, C7: 10uF, Capacitor_SMD:C_0805_2012Metric, symbol Device:C
- removed C39, C5: 100nF, Capacitor_SMD:C_0603_1608Metric, symbol Device:C
- removed C40, C6: 10nF, Capacitor_SMD:C_0603_1608Metric, symbol Device:C
- removed L1: 4.7uH, Inductor_SMD:L_Taiyo-Yuden_MD-3030, symbol Device:L
- removed Q1, Q2: 2N7002, Package_TO_SOT_SMD:SOT-23, symbol Transistor_FET:2N7002
- removed Q3: BSS138W, PCM_JLCPCB:Q_SOT-323, symbol PCM_JLCPCB-Transistors:NMOS,BSS138W
- removed S1, S2, S3: ~, footprints:CapTouchButton, symbol parts:CapTouchPad
- removed U1: TPS61222DCK, Package_TO_SOT_SMD:Texas_R-PDSO-G6, symbol Regulator_Switching:TPS61222DCK
- removed U5: LPC804M101JHI33, Package_DFN_QFN:QFN-32-1EP_5x5mm_P0.5mm_EP3.7x3.7mm, symbol parts:LPC804M101JHI33
- added C51, C52: 1uF, Capacitor_SMD:C_0805_2012Metric, symbol Device:C
- added Q5: BSS138W, Package_TO_SOT_SMD:SOT-23W, symbol Transistor_FET:BSS138
- added TP10, TP8, TP9: TestPoint_Small, TestPoint:TestPoint_Pad_D2.0mm, symbol Connector:TestPoint_Small
- C1, C2: $/1,10,100 0.110,0.042,0.027 -> (none)
- C3, C4, C46: $/1,10,100 0.170,0.068,0.044 -> (none)
- Q4: value BSS138 -> BSS138W; footprint Package_TO_SOT_SMD:SOT-23 -> Package_TO_SOT_SMD:SOT-23W; LCSC Part # (none) -> C28646265
Connections:
- net CAPT_X0 is gone; now on net SW1: TP6.1
- net CAPT_X1 is gone; now on net SW2: TP2.1
- net CAPT_X2 is gone; now on net SW3: TP7.1
- net +3V3: now also C2.2, J4.3 (Pin_3), C52.1
- net +5V: now also C48.2, D7.1 (K), J4.1 (Pin_1), U15.4 (VOUT), C51.1; no longer C2.2
- net +BATT: now also C1.2, L4.1
- net GND: now also C47.2, C49.2, C50.2, J4.2 (Pin_2), J4.4 (Pin_4), SW1.1, SW2.1, SW3.1, C51.2, C52.2
- net LEDs/CKI: now also Q5.3 (D), TP9.1
- net LEDs/SDI: now also Q4.3 (D), TP10.1
- net SPI0_MOSI: no longer R3.2, U3.17 (PA7)
- net SPI1_MISO: now also TP8.1
- net SPI1_SCK: now also Q5.1 (G), Q5.2 (S)
- net SPI1_MOSI: now reaches Q4.1 (G)
- net SPI1_MOSI: now also Q4.2 (S), R3.2, U3.17 (PA7)
- net CAPT_YH: no longer names the net of C32.1
- net CAPT_YL: no longer names the net of C32.2
- no-connect marks 34 -> 21
Other:
- note added: "3V3 LDO"
- note removed: "ACMP_I4"
- note removed: "ADC_10"
- moved on the sheet: C1, C3, C41, C42, C43, C45, C47, C48, C49, C50, D7, H1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

Commit message: Prelim connector pinout defined.  Re-annotated all parts
Parts:
- removed J4, J5: Conn_01x10, Connector_PinHeader_2.54mm:PinHeader_1x10_P2.54mm_Vertical, symbol Connector_Generic:Conn_01x10
- added J3, J4: Conn_01x12, Connector_PinSocket_2.54mm:PinSocket_1x12_P2.54mm_Vertical, symbol Connector_Generic:Conn_01x12
- added NT1: NetTie_2, NetTie:NetTie-2_SMD_Pad0.5mm, symbol Device:NetTie_2
- added R3, R6: 10K, Resistor_SMD:R_0805_2012Metric, symbol Device:R
- renumbered C43 to C10, C45 to C11, C46 to C12, C49 to C13, C47 to C14, C50 to C15, C32 to C16, C48 to C2, C52 to C5, C51 to C6, C2 to C7, C41 to C8, C42 to C9, D7 to D1, H2 to H1, H1 to H2, H4 to H3, H3 to H4, J3 to J5, L4 to L1, Q5 to Q1, Q4 to Q2, R5 to R1, R2 to R10, R1 to R11, R6 to R2, R3 to R4, R4 to R5, R11 to R7, R10 to R8, R12 to R9, SW2 to SW1, SW1 to SW2, TP3 to TP1, TP7 to TP10, TP4 to TP2, TP1 to TP3, TP5 to TP4, TP9 to TP5, TP8 to TP6, TP10 to TP7, TP2 to TP8, TP6 to TP9, U2 to U1, U15 to U2
Connections:
- net +3V3: now also J3.3 (Pin_3), J3.4 (Pin_4), R3.1
- net +5V: now also J3.1 (Pin_1)
- net +BATT: now also NT1.1; no longer C1.2, L1.1, TP4.1, U3.10 (PA0)
- net GND: now also J3.10 (Pin_10), J3.2 (Pin_2), J3.5 (Pin_5), J3.7 (Pin_7), J4.1 (Pin_1), J4.5 (Pin_5), J4.8 (Pin_8), R6.2
- net GPIO_EXTI10: now also J3.12 (Pin_12)
- net I2C1_SCL: now also J3.8 (Pin_8)
- net I2C1_SDA: now also J3.9 (Pin_9)
- net SPI2_MISO: now also J4.10 (Pin_10)
- net SPI2_MOSI: now also J4.9 (Pin_9)
- net SPI2_NSS: now also J4.12 (Pin_12)
- net SPI2_SCK: now also J4.11 (Pin_11)
- net SWCLK: now also J4.3 (Pin_3)
- net SWDIO: now also J4.4 (Pin_4)
- net USART1_RX: now also J4.6 (Pin_6)
- net USART1_TX: now also J4.7 (Pin_7)
- net nRST: now also J4.2 (Pin_2), R3.2
- net PB2: now reaches U3.20 (PB2)
- net PB2: now also J3.11 (Pin_11)
- net BOOT0: now reaches U3.44 (BOOT0)
- net BOOT0: now also J3.6 (Pin_6), R6.1
- new net ADC_IN0: C1.2, L1.1, NT1.2, TP4.1, U3.10 (PA0)
Other:
- moved on the sheet: C10, C11, C12, C13, C14, C15, C16, C5, C6, C7, C8, C9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
