File: nfc.kicad_sch (KiCad schematic)
At the start: 31 parts, among them U4 ST25R3911B-AQFT, Y1 27.12MHz

Commit message: Prelim connector pinout defined.  Re-annotated all parts
Parts:
- renumbered C8 to C22, C9 to C23, C10 to C24, C11 to C25, C12 to C26, C13 to C27, C14 to C28, C15 to C29, C16 to C30, C17 to C31, C18 to C32, C19 to C33, C20 to C34, C21 to C35, C22 to C36, C23 to C37, C24 to C38, C25 to C39, C26 to C40, C33 to C41, C34 to C42, C35 to C43, C36 to C44, C37 to C45, R7 to R12, R8 to R13, U4 to U9

Commit message: Added I2C resistors to schematic, cleaned up unused parts and started layout
Parts:
- renumbered R12 to R14, R13 to R15
Changed lines of the file:
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@@
 		(on_board yes)
 		(dnp no)
-		(property "Reference" "#PWR0113"
+		(property "Reference" "#PWR?"
 			(at 200.66 118.11 0)
 			(effects
@@
 			(project "lmc_media_blitz"
 				(path "/b87eb037-3127-4116-a225-5eb939725614/1dee4cad-e641-4e05-a4e5-3096da974ea0"
-					(reference "#PWR0113")
+					(reference "#PWR?")
 					(unit 1)
 				)
@@
 		(on_board yes)
 		(dnp no)
-		(property "Reference" "R12"
+		(property "Reference" "R14"
 			(at 227.33 95.758 90)
 			(effects
@@
 			(project "lmc_media_blitz"
 				(path "/b87eb037-3127-4116-a225-5eb939725614/1dee4cad-e641-4e05-a4e5-3096da974ea0"
-					(reference "R12")
+					(reference "R14")
 					(unit 1)
 				)
@@
 		(on_board yes)
 		(dnp no)
-		(property "Reference" "#PWR0114"
+		(property "Reference" "#PWR?"
 			(at 128.27 52.07 0)
 			(effects
@@
 			(project "lmc_media_blitz"
 				(path "/b87eb037-3127-4116-a225-5eb939725614/1dee4cad-e641-4e05-a4e5-3096da974ea0"
-					(reference "#PWR0114")
+					(reference "#PWR?")
 					(unit 1)
 				)
@@
 		(on_board yes)
 		(dnp no)
-		(property "Reference" "#PWR0116"
+		(property "Reference" "#PWR?"
 			(at 91.44 100.33 0)
 			(effects
@@
 			(project "lmc_media_blitz"
 				(path "/b87eb037-3127-4116-a225-5eb939725614/1dee4cad-e641-4e05-a4e5-3096da974ea0"
-					(reference "#PWR0116")
+					(reference "#PWR?")
 					(unit 1)
 				)
@@
 		(on_board yes)
 		(dnp no)
-		(property "Reference" "#PWR0119"
+		(property "Reference" "#PWR?"
 			(at 214.63 146.05 0)
 			(effects
@@
 			(project "lmc_media_blitz"
 				(path "/b87eb037-3127-4116-a225-5eb939725614/1dee4cad-e641-4e05-a4e5-3096da974ea0"
-					(reference "#PWR0119")
+					(reference "#PWR?")
 					(unit 1)
 				)
@@
 		(on_board yes)
 		(dnp no)
-		(property "Reference" "#PWR0118"
+		(property "Reference" "#PWR?"
 			(at 116.84 120.65 0)
 			(effects
@@
 			(project "lmc_media_blitz"
 				(path "/b87eb037-3127-4116-a225-5eb939725614/1dee4cad-e641-4e05-a4e5-3096da974ea0"
-					(reference "#PWR0118")
+					(reference "#PWR?")
 					(unit 1)
 				)
@@
 		(on_board yes)
 		(dnp no)
-		(property "Reference" "#PWR0112"
+		(property "Reference" "#PWR?"
 			(at 172.72 118.11 0)
 			(effects
@@
 			(project "lmc_media_blitz"
 				(path "/b87eb037-3127-4116-a225-5eb939725614/1dee4cad-e641-4e05-a4e5-3096da974ea0"
-					(reference "#PWR0112")
+					(reference "#PWR?")
 					(unit 1)
 				)
@@
 		(on_board yes)
 		(dnp no)
-		(property "Reference" "#PWR0117"
+		(property "Reference" "#PWR?"
 			(at 77.47 115.57 0)
 			(effects
@@
 			(project "lmc_media_blitz"
 				(path "/b87eb037-3127-4116-a225-5eb939725614/1dee4cad-e641-4e05-a4e5-3096da974ea0"
-					(reference "#PWR0117")
+					(reference "#PWR?")
 					(unit 1)
 				)
@@
 		(on_board yes)
 		(dnp no)
-		(property "Reference" "R13"
+		(property "Reference" "R15"
 			(at 227.33 116.078 90)
 			(effects
@@
 			(project "lmc_media_blitz"
 				(path "/b87eb037-3127-4116-a225-5eb939725614/1dee4cad-e641-4e05-a4e5-3096da974ea0"
-					(reference "R13")
+					(reference "R15")
 					(unit 1)
 				)
@@
 		(on_board yes)
 		(dnp no)
-		(property "Reference" "#PWR0124"
+		(property "Reference" "#PWR?"
 			(at 110.49 52.07 0)
 			(effects
@@
 			(project "lmc_media_blitz"
 				(path "/b87eb037-3127-4116-a225-5eb939725614/1dee4cad-e641-4e05-a4e5-3096da974ea0"
-					(reference "#PWR0124")
+					(reference "#PWR?")
 					(unit 1)
 				)
@@
 		(on_board yes)
 		(dnp no)
-		(property "Reference" "#PWR0121"
+		(property "Reference" "#PWR?"
 			(at 231.14 87.63 0)
 			(effects
@@
 			(project "lmc_media_blitz"
 				(path "/b87eb037-3127-4116-a225-5eb939725614/1dee4cad-e641-4e05-a4e5-3096da974ea0"
-					(reference "#PWR0121")
+					(reference "#PWR?")
 					(unit 1)
 				)
@@
 		(on_board yes)
 		(dnp no)
-		(property "Reference" "#PWR0122"
+		(property "Reference" "#PWR?"
 			(at 140.97 36.83 0)
 			(effects
@@
 			(project "lmc_media_blitz"
 				(path "/b87eb037-3127-4116-a225-5eb939725614/1dee4cad-e641-4e05-a4e5-3096da974ea0"
-					(reference "#PWR0122")
+					(reference "#PWR?")
 					(unit 1)
 				)
@@
 		(on_board yes)
 		(dnp no)
-		(property "Reference" "#PWR0123"
+		(property "Reference" "#PWR?"
 			(at 99.06 36.83 0)
 			(effects
@@
 			(project "lmc_media_blitz"
 				(path "/b87eb037-3127-4116-a225-5eb939725614/1dee4cad-e641-4e05-a4e5-3096da974ea0"
-					(reference "#PWR0123")
+					(reference "#PWR?")
 					(unit 1)
 				)
@@
 		(on_board yes)
 		(dnp no)
-		(property "Reference" "#PWR0120"
+		(property "Reference" "#PWR?"
 			(at 207.01 71.12 0)
 			(effects
@@
 			(project "lmc_media_blitz"
 				(path "/b87eb037-3127-4116-a225-5eb939725614/1dee4cad-e641-4e05-a4e5-3096da974ea0"
-					(reference "#PWR0120")
+					(reference "#PWR?")
 					(unit 1)
 				)
@@
 		(on_board yes)
 		(dnp no)
-		(property "Reference" "#PWR0115"
+		(property "Reference" "#PWR?"
 			(at 157.48 85.09 0)
 			(effects
@@
 			(project "lmc_media_blitz"
 				(path "/b87eb037-3127-4116-a225-5eb939725614/1dee4cad-e641-4e05-a4e5-3096da974ea0"
-					(reference "#PWR0115")
+					(reference "#PWR?")
 					(unit 1)
 				)
